Commit message: fiix end-effector offset

File: ft_tools_examples/config/effector.urdf.xacro (robot description, xacro)
@@ -4,5 +4,5 @@
   <link name="${prefix}ft_sensor"/>
   <joint name="${prefix}joint_tool0-ft_sensor" type="fixed">
-      <origin rpy="0 0 0" xyz="0 0 0.025"/>
+      <origin rpy="0 0 0" xyz="0 0 0.026"/>
       <parent link="${prefix}${parent}"/>
       <child link="${prefix}ft_sensor"/>

Commit message: add interaction frame

File: ft_tools_examples/config/effector.urdf.xacro (robot description, xacro)
@@ -9,4 +9,11 @@
       <axis xyz="0 0 0"/>
   </joint>
+  <link name="${prefix}interaction_point"/>
+  <joint name="${prefix}ft_sensor-interaction_point" type="fixed">
+      <origin rpy="0 0 0" xyz="0 0 0.1"/>
+      <parent link="${prefix}ft_sensor"/>
+      <child link="${prefix}interaction_point"/>
+      <axis xyz="0 0 0"/>
+  </joint>
   </xacro:macro>
 </robot>
